File: SEN00001/SEN00001.brd (EAGLE design)
At the start: 47 x 50.5 mm, 14 parts, among them U1 QRE1113, U2 QRE1113, U3 QRE1113

Commit message: Updated Description
Updated layout and schematic. Updated readme file and added pdf versions
of the schematic and board
Parts:
- added CC_TEXT1: CREATIVE_COMMONS, SparkFun-Aesthetics:CREATIVE_COMMONS
Other:
- board text added: "B. Carrizales"
Changed lines of the file:
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@@
 <wire x1="46.97" y1="50.47" x2="0" y2="50.47" width="0" layer="20"/>
 <wire x1="0" y1="50.47" x2="0" y2="0" width="0" layer="20"/>
+<text x="30.48" y="-10.16" size="1.778" layer="51">B. Carrizales</text>
 </plain>
 <attributes>
@@
 <element name="STANDOFF3" library="SparkFun-Electromechanical" package="STAND-OFF" value="STAND-OFF" x="40.64" y="6.35"/>
 <element name="STANDOFF4" library="SparkFun-Electromechanical" package="STAND-OFF" value="STAND-OFF" x="40.64" y="44.45"/>
+<element name="CC_TEXT1" library="SparkFun-Aesthetics" package="CREATIVE_COMMONS" value="CREATIVE_COMMONS" x="5.08" y="-10.16"/>
 </elements>
 <signals>
