File: SEN00001/SEN00001.sch (EAGLE design)
At the start: 14 parts, among them U1 QRE1113, U2 QRE1113, U3 QRE1113

Commit message: Updated Description
Updated layout and schematic. Updated readme file and added pdf versions
of the schematic and board
Parts:
- added CC_TEXT1: CREATIVE_COMMONS, SparkFun-Aesthetics:CREATIVE_COMMONS
Other:
- note added: "B. Carrizales"
Changed lines of the file:
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@@
 <part name="STANDOFF3" library="SparkFun-Electromechanical" deviceset="STAND-OFF" device=""/>
 <part name="STANDOFF4" library="SparkFun-Electromechanical" deviceset="STAND-OFF" device=""/>
+<part name="CC_TEXT1" library="SparkFun-Aesthetics" deviceset="CREATIVE_COMMONS" device=""/>
 </parts>
 <sheets>
@@
 <text x="127" y="-105.41" size="1.778" layer="91">1 of 1</text>
 <text x="127" y="-98.298" size="1.778" layer="91">0</text>
+<text x="-22.86" y="-104.14" size="1.778" layer="91">B. Carrizales</text>
 </plain>
 <instances>
@@
 <instance part="STANDOFF3" gate="G$1" x="-119.38" y="-60.96"/>
 <instance part="STANDOFF4" gate="G$1" x="-119.38" y="-55.88"/>
+<instance part="CC_TEXT1" gate="G$1" x="-35.56" y="-104.14"/>
 </instances>
 <busses>
